File: Hardware/MicroMouse.kicad_pcb (KiCad board)
At the start: 2 copper layers, 65 x 40 mm, 80 parts, among them J1 TSW-106-25-S-S-RA, J2 B2B-PH-K-S(LF)(SN), J3 Conn_01x04_Male, J4 B5B-XH-A(LF)(SN), J5 B5B-XH-A(LF)(SN), Q1 NXV75UPR, SW1 SPST, SW2 SPST, SW3 SPST, SW4 SPST, SW6 SPST, SW7 SPST, SW8 SPST, U1 ADP1612, U2 PIC16F886-E_SO, U3 ULN2803ADW, U4 74LVC1G332GV-Q100H, U5 ADCMP393ARZ, U6 TCRT1000, U7 TCRT1000, U8 TCRT1000, Y1 32.768KHZ

Commit message: Layout
Parts:
- added C9: 0.1uF, Micro-Footprint:CAP0603, B.Cu at (97.6, 99.9)
- C10, C12, FB1, R12, R13, R7, R8: moved to B.Cu
- moved R8 70.5 mm to (124.3, 80.5)
- moved FB1 61.9 mm to (113.8, 95.3), turned to 90 degrees
- moved R7 58.1 mm to (124.3, 81.8)
- moved C12 47.0 mm to (115.2, 95.2), turned to 90 degrees
- moved R24 39.4 mm to (79.3, 85.1), turned to 180 degrees
- moved R12 38.4 mm to (110.4, 86.2)
- moved R25 38.3 mm to (79.3, 86.4), turned to 180 degrees
- moved C10 35.0 mm to (97.6, 98.6), turned to 180 degrees
- moved R13 30.5 mm to (110.4, 87.6), turned to 180 degrees
- moved D3 16.3 mm to (59.9, 107.1)
- moved D5 12.6 mm to (55.2, 111.6)
- moved U7 6.00 mm to (71.0, 100.0)
- moved U8 6.00 mm to (71.0, 80.0)
- moved C7 4.30 mm to (116.5, 95.2), turned to 90 degrees
- moved D4 3.39 mm to (69.7, 118.1)
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Routing:
- net GND: track 0.00 -> 147.9 mm, vias 0 -> 9
- net +5P: track 0.00 -> 120.0 mm, vias 0 -> 6
- net /RW2: track 0.00 -> 60.2 mm
- net /CL2: track 0.00 -> 41.7 mm
- net /RW1: track 0.00 -> 39.4 mm
- net /CL3: track 0.00 -> 36.2 mm
- net /Vpp: track 0.00 -> 31.6 mm
- net /Aux: track 0.00 -> 30.5 mm, vias 0 -> 1
- net VCC: track 0.00 -> 27.1 mm, vias 0 -> 5
- net +5V: track 0.00 -> 22.5 mm
- net Net-(R12-Pad1): track 0.00 -> 21.3 mm
- net Net-(U2-Pad10): track 0.00 -> 17.7 mm, vias 0 -> 1
- net Net-(C5-Pad1): track 0.00 -> 13.6 mm, vias 0 -> 4
- net Net-(U2-Pad9): track 0.00 -> 13.0 mm, vias 0 -> 1
- net Net-(U2-Pad5): track 0.00 -> 12.9 mm, vias 0 -> 1
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
Commit message: Update Layout
Parts:
- removed C11: 1uF, Micro-Footprint:CAP0603
- removed the C9 at (83.1, 124.0)
- C13, C15, C16, R18, Y1: moved to B.Cu
- moved R11 51.1 mm to (86.8, 91.0), turned to 180 degrees
- moved R21 51.0 mm to (69.8, 84.3)
- moved R22 48.3 mm to (73.3, 73.7), turned to 270 degrees
- moved Y1 47.8 mm to (114.5, 103.7), turned to 180 degrees
- moved D6 44.1 mm to (76.8, 79.2)
- moved R14 40.2 mm to (70.3, 94.8)
- moved R17 40.2 mm to (77.1, 80.7), turned to 180 degrees
- moved C13 39.8 mm to (94.7, 89.8)
- moved R15 38.2 mm to (69.8, 85.7), turned to 180 degrees
- moved C4 36.1 mm to (94.8, 86.6), turned to 270 degrees
- moved R16 35.1 mm to (75.7, 101.3), turned to 180 degrees
- moved D4 30.6 mm to (86.5, 92.5)
- moved R6 28.2 mm to (93.5, 86.6), turned to 270 degrees
- moved C16 25.9 mm to (114.1, 106.2), turned to 90 degrees
- moved C15 25.2 mm to (115.5, 106.2), turned to 90 degrees
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Routing:
- net /RHT: track 0.00 -> 44.6 mm, vias 0 -> 1
- net /LFT: track 0.00 -> 39.8 mm, vias 0 -> 3
- net /FRT: track 0.00 -> 26.1 mm, vias 0 -> 2
- net GND: track 147.9 -> 130.4 mm, vias 9 -> 11
- net Net-(R20-Pad2): track 0.00 -> 6.47 mm
- net Net-(C16-Pad2): track 0.00 -> 4.61 mm
- net Net-(C15-Pad2): track 0.00 -> 3.90 mm
- net Net-(R21-Pad1): track 0.00 -> 3.43 mm
- net Net-(R18-Pad2): track 0.00 -> 3.15 mm
- net Net-(R22-Pad2): track 0.00 -> 2.72 mm
- net Net-(D2-Pad2): track 2.66 -> 5.34 mm
- net Net-(J3-Pad3): track 0.00 -> 2.41 mm
- net Net-(J3-Pad4): track 0.00 -> 2.35 mm
- net Net-(R15-Pad2): track 0.00 -> 1.79 mm
- net +5P: track 120.0 -> 121.8 mm
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
Commit message: Update Layout
Parts:
- moved U7 1.00 mm to (72.0, 101.0)
- moved R19 0.85 mm to (73.8, 105.9)
- moved R22 0.73 mm to (73.5, 74.4)
Routing:
- net +5P: track 121.8 -> 239.3 mm, vias 6 -> 15
- net GND: track 130.4 -> 235.9 mm, vias 11 -> 18
- net /RW1: track 39.4 -> 93.6 mm, vias 0 -> 1
- net /RW2: track 58.9 -> 108.9 mm, vias 0 -> 2
- net Net-(J3-Pad4): track 2.35 -> 45.9 mm
- net /CL1: track 0.00 -> 42.7 mm, vias 0 -> 2
- net Net-(D3-Pad1): track 0.00 -> 40.7 mm, vias 0 -> 1
- net Net-(RV2-Pad2): track 0.00 -> 22.8 mm, vias 0 -> 1
- net Net-(U2-Pad21): track 0.00 -> 17.0 mm, vias 0 -> 2
- net Net-(R22-Pad2): track 2.72 -> 14.1 mm
- net Net-(RV1-Pad2): track 0.00 -> 9.28 mm, vias 0 -> 1
- net Net-(RV3-Pad2): track 0.00 -> 5.96 mm
- net /RHT: track 44.6 -> 40.9 mm
- net Net-(R20-Pad2): track 6.47 -> 3.05 mm
- net Net-(R19-Pad1): track 0.00 -> 2.08 mm
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
Commit message: Layout Update
Parts:
- moved C14 0.50 mm to (86.5, 94.0)
- moved R11 0.34 mm to (86.5, 91.0)
Routing:
- net Net-(J3-Pad3): track 2.41 -> 52.6 mm
- net GND: track 235.9 -> 260.9 mm, vias 18 -> 16
- net Net-(R20-Pad2): track 3.05 -> 28.0 mm, vias 0 -> 1
- net /FRT: track 26.5 -> 43.5 mm
- net /CL1: track 42.7 -> 57.7 mm, vias 2 -> 1
- net +5P: track 239.3 -> 252.4 mm, vias 15 -> 11
- net Net-(D3-Pad1): track 40.7 -> 30.5 mm
- net Net-(RV1-Pad2): track 9.28 -> 1.15 mm, vias 1 -> 0
- net Net-(J3-Pad4): track 45.9 -> 41.5 mm
- net /RW2: track 108.9 -> 112.4 mm
- net Net-(R14-Pad1): track 0.00 -> 2.49 mm
- net /CL3: track 36.2 -> 38.1 mm
- net /CL2: track 41.7 -> 40.6 mm
- net Net-(RV2-Pad2): track 22.8 -> 23.9 mm, vias 1 -> 0
- net Net-(U2-Pad21): track 17.0 -> 16.3 mm
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
Commit message: Add files via upload
Routing:
- net /CL1: track 57.7 -> 77.3 mm, vias 1 -> 3
- net Net-(RV2-Pad2): track 23.9 -> 36.7 mm
- net Net-(D3-Pad1): track 30.5 -> 40.6 mm
- net GND: track 260.9 -> 269.0 mm

Commit message: Update layout
Parts:
- moved C13 4.57 mm to (90.6, 91.8), turned to 90 degrees
- moved C8 2.18 mm to (124.6, 99.9), turned to 0 degrees
Routing:
- net GND: track 269.0 -> 352.9 mm, vias 16 -> 18
- net Net-(R15-Pad2): track 1.79 -> 82.4 mm, vias 0 -> 1
- net Net-(RV3-Pad2): track 5.96 -> 76.2 mm, vias 0 -> 1
- net Net-(R22-Pad2): track 14.1 -> 79.0 mm, vias 0 -> 1
- net /CL3: track 38.1 -> 59.8 mm, vias 0 -> 2
- net /RW1: track 93.6 -> 113.8 mm, vias 1 -> 3
- net Net-(RV2-Pad2): track 36.7 -> 18.5 mm
- net /CL2: track 40.6 -> 56.8 mm, vias 0 -> 2
- net /RW2: track 112.4 -> 127.2 mm
- net Net-(RV1-Pad2): track 1.15 -> 14.1 mm, vias 0 -> 1
- net /CL1: track 77.3 -> 89.2 mm, vias 3 -> 4
- net VCC: track 27.1 -> 36.7 mm
- net +5P: track 252.4 -> 259.9 mm, vias 11 -> 14
- net Net-(J2-Pad1): track 6.95 -> 13.2 mm
- net Net-(R12-Pad1): track 22.0 -> 28.0 mm
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Other:
- net class Default: clearance 0.2 -> 0.127; trace_width 0.25 -> 0.127; via_dia 0.8 -> 0.6; via_drill 0.4 -> 0.3
- net class Setup1 added: clearance 0.127, trace_width 0.127, via_dia 0.6, via_drill 0.3
- rule trace_clearance: 0.2 -> 0.127
- rule trace_min: 0.2 -> 0.127
- rule via_min_size: 0.4 -> 0.25
